File: electronics/star-track.kicad_sch (KiCad schematic)
At the start: 27 parts, among them J1 XT60 battery, J2 XT60 charge, J3 Joystick, J4 AZ motor, J5 ALT motor, SW1 Main switch, SW2 E-stop (NC), SW3 Push button, SW4 Push button, SW5 Push button, U1 L7805CV

Commit message: Drop charging circuit; add hand unit, LEDs and buzzer
- Schematic: female XT60 input for the battery or a lab supply, no
  charge socket. Joystick and buttons moved to a hand unit on an 8-pin
  socket, with 100 nF filters on the joystick lines. Red and blue LEDs
  (GPIO15, GPIO16) and a buzzer driven by an NPN transistor (GPIO21).
- docs/architecture.md: hand unit, feedback, power input and lab supply,
  notes on charging LiFePO4 with a lead-acid charger.
- docs/mechanics.md, docs/3d: case face with E-stop, LEDs, buzzer and
  main switch, sockets underneath; packed head size updated.

Co-Authored-By: Claude Opus 5.5 <noreply@anthropic.com>
Claude-Session: https://claude.ai/code/session_019gYbrjmddARBSj5u2J2ySh
Parts:
- removed A3: TMC2209 ALT, symbol star-track:TMC2209_module
- removed J2: XT60 charge, symbol Connector_Generic:Conn_01x02
- added BZ1: Buzzer, symbol Device:Buzzer
- added C8, C9: 100nF, symbol Device:C
- added D2: 1N4148, symbol Device:D
- added D3: red, symbol Device:LED
- added D4: blue, symbol Device:LED
- added J2: Hand unit, 8 pins, symbol Connector_Generic:Conn_01x08
- added Q1: BC547, symbol Device:Q_NPN_BCE
- added R5, R7: 1k, symbol Device:R
- added R6: 10k, symbol Device:R
- added R8: 220, symbol Device:R
- added SW2: E-stop (NC), symbol Switch:SW_Push_Open
- A3: renamed from SW2; value E-stop (NC) -> TMC2209 ALT; symbol Switch:SW_Push_Open -> star-track:TMC2209_module
- J1: value XT60 battery -> XT60 female
- J3: value Joystick -> Joystick module
Connections:
- net +12V: now also A3.9 (VM)
- net +3V3: now also A3.15 (VIO), A3.2 (MS1), J2.2 (Pin_2)
- net +5V: now also BZ1.1 (+), D2.1 (K)
- net ALT_DIR: now also A3.8 (DIR)
- net ALT_STEP: now also A3.7 (STEP)
- net BTN1: now also J2.6 (Pin_6)
- net BTN2: now also J2.7 (Pin_7)
- net BTN3: now also J2.8 (Pin_8)
- net DRV_EN: now also A3.1 (EN), SW2.2 (B); no longer A3.2 (B)
- net DRV_UART: now also A3.4 (PDN_UART)
- net EN_OUT: now also SW2.1 (A); no longer A3.1 (A)
- net GND: now also A3.10 (GND), A3.16 (GND), A3.3 (MS2), C8.2, C9.2, D3.1 (K), D4.1 (K), J2.1 (Pin_1), Q1.3 (E), R6.2
- net JOY_SW: now also J2.5 (Pin_5)
- net JOY_X: now also C8.1, J2.3 (Pin_3)
- net JOY_Y: now also C9.1, J2.4 (Pin_4)
- net at J5.4 (Pin_4): now also A3.11 (2B)
- net at J5.3 (Pin_3): now also A3.12 (2A)
- net at J5.1 (Pin_1): now also A3.13 (1A)
- net at J5.2 (Pin_2): now also A3.14 (1B)
- net BUZZER: now reaches A1.40 (GPIO21)
- net BUZZER: now also R5.1
- net LED_RED: now reaches A1.8 (GPIO15)
- net LED_RED: now also R7.1
- net LED_BLUE: now reaches A1.9 (GPIO16)
- net LED_BLUE: now also R8.1
- new net: Q1.1 (B), R5.2, R6.1
- new net: BZ1.2 (-), D2.2 (A), Q1.2 (C)
- new net: D4.2 (A), R8.2
- new net: D3.2 (A), R7.2
- no-connect marks 24 -> 21
Other:
- note added: "1. Supply, controller and drivers are all on the L: no cable crosses the azimuth joint. 2. +12V is the switched supply rail (12.0-14.6 V). It feeds the drivers and U1. 3. TMC2209 modules: VIO at 3.3 V (ESP32 logic level); motor current is set over UART. The header pin order differs between makers: wire by pin name. 4. Motor connectors: pins 1-2 = one coil, pins 3-4 = the other coil. 5. A1 pin num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"
- note added: "E-stop (on the case)"
- note added: "GPIO high = LED on. PWM sets the brightness."
- note added: "Hand unit (on the cable)"
- note added: "Hand-unit socket (on the case)"
- note added: "J1: female XT60 on the case, for the battery (LiFePO4 12.8 V 6 Ah with BMS) or a lab supply (12-14 V, current limit about 2 A). The battery is charged off the mount."
- note added: "LEDs and buzzer (on the case)"
- note added: "Power input, fuse, main switch"
- note removed: "1. Battery, controller and drivers are all on the L: no cable crosses the azimuth joint. 2. +12V is the switched battery rail (12.0-14.6 V). It feeds the drivers and U1. 3. TMC2209 modules: VIO at 3.3 V (ESP32 logic level); motor current is set over UART. The header pin order differs between makers: wire by pin name. 4. Motor connectors: pins 1-2 = one coil, pins 3-4 = the other coil. 5. A1 pin n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"
- note removed: "14.6 V LiFePO4 charger. Charging works with SW1 off."
- note removed: "Battery, fuse, main switch"
- note removed: "LiFePO4 12.8 V 6 Ah with BMS"
- note removed: "Manual controls"

Commit message: Simplify the circuit to the parts that are needed
- Resettable breaker switch replaces the fuse and the main switch.
- TMC2209 drivers in standalone mode (1/64 microsteps with MS1/MS2,
  current from the Vref potentiometer): no UART resistor or wires.
- Buzzer directly on GPIO21, without the transistor stage.
- Removed the bulk and regulator capacitors, the battery voltage
  divider and the joystick filter capacitors.
- docs/architecture.md: why the remaining parts are needed, and a
  "Left out" table with what each removed part would add.

Co-Authored-By: Claude Opus 5.5 <noreply@anthropic.com>
Claude-Session: https://claude.ai/code/session_019gYbrjmddARBSj5u2J2ySh
Parts:
- removed A2: TMC2209 AZ, symbol star-track:TMC2209_module
- removed C1: 470µF 25V, symbol Device:C_Polarized
- removed C2: 330nF, symbol Device:C
- removed C3, C5, C8, C9: 100nF, symbol Device:C
- removed C4: 47µF 10V, symbol Device:C_Polarized
- removed D2: 1N4148, symbol Device:D
- removed F1: 5 A, symbol Device:Fuse
- removed J2: Hand unit, 8 pins, symbol Connector_Generic:Conn_01x08
- removed Q1: BC547, symbol Device:Q_NPN_BCE
- removed R1: 100k, symbol Device:R
- removed R4, R5: 1k, symbol Device:R
- removed R6: 10k, symbol Device:R
- removed SW1: Main switch, symbol Switch:SW_SPST
- added C6: 100µF 25V, symbol Device:C_Polarized
- added CB1: Breaker switch, symbol Device:CircuitBreaker_1P
- A2: renamed from R2; value 22k -> TMC2209 AZ; symbol Device:R -> star-track:TMC2209_module
- J2: renamed from C6; value 100µF 25V -> Hand unit, 8 pins; symbol Device:C_Polarized -> Connector_Generic:Conn_01x08
Connections:
- net +12V: now also A2.9 (VM), C6.1, CB1.2; no longer J2.1
- net +3V3: now also A2.15 (VIO), A2.3 (MS2), A3.3 (MS2), J2.2 (Pin_2); no longer A3.2 (MS1)
- net +5V: no longer BZ1.1 (+)
- net AZ_DIR: now also A2.8 (DIR)
- net AZ_STEP: now also A2.7 (STEP)
- net BTN1: now also J2.6 (Pin_6)
- net BTN2: now also J2.7 (Pin_7)
- net BTN3: now also J2.8 (Pin_8)
- net BUZZER: now also BZ1.1 (+)
- net DRV_EN: now also A2.1 (EN)
- net GND: now also A2.10 (GND), A2.16 (GND), A3.2 (MS1), BZ1.2 (-), J2.1 (Pin_1), C6.2; no longer A3.3 (MS2), J2.2
- net JOY_SW: now also J2.5 (Pin_5)
- net JOY_X: now also J2.3 (Pin_3)
- net JOY_Y: now also J2.4 (Pin_4)
- net at J4.4 (Pin_4): now also A2.11 (2B)
- net at J4.3 (Pin_3): now also A2.12 (2A)
- net at J4.1 (Pin_1): now also A2.13 (1A)
- net at J4.2 (Pin_2): now also A2.14 (1B)
- net at J1.1 (Pin_1): now also CB1.1
- net DRV_UART: no longer names the net of A3.4 (PDN_UART)
- net DRV_UART: no longer A1.11 (GPIO18)
- net UART_TX: no longer names the net of A1.10 (GPIO17)
- net VBAT_SENSE: no longer names the net of A1.4 (GPIO4)
- net VBAT_SENSE: no longer A2.1
- no-connect marks 21 -> 26
Other:
- note added: "1. Supply, controller and drivers are all on the L: no cable crosses the azimuth joint. 2. +12V: 12.0-14.6 V from the battery or a lab supply. It feeds the drivers and U1. 3. TMC2209 header pin order differs between makers: wire by pin name. VIO at 3.3 V (ESP32 logic level). 4. Motor connectors: pins 1-2 one coil, 3-4 the other. 5. A1 pins: 1-22 = header J1, 23-44 = header J3. 6. Hand unit on an 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"
- note added: "GPIO high = LED or buzzer on. PWM sets the LED brightness, or the tone of a passive buzzer."
- note added: "Hand-unit socket (case)"
- note added: "J1: female XT60 on the case, for the battery (LiFePO4 12.8 V 6 Ah with BMS) or a lab supply (12-14 V, current limit about 2 A). The battery is charged off the mount. CB1: resettable breaker switch, 3-5 A, rated for DC."
- note added: "Power input and breaker switch"
- note added: "Standalone mode, no UART: MS1 = GND, MS2 = 3V3 gives 1/64 microsteps. Motor current: potentiometer (Vref) on each module. C6, C7 must sit close to the VM pins: they absorb the motor voltage spikes."
- note added: "U1 on a small TO-220 heatsink (tab = GND), about 1 W. Place it near C6/C7, which also serve as its input capacitors. D1 stops U1 and the board's USB 5 V from feeding each other."
- note removed: "1. Supply, controller and drivers are all on the L: no cable crosses the azimuth joint. 2. +12V is the switched supply rail (12.0-14.6 V). It feeds the drivers and U1. 3. TMC2209 modules: VIO at 3.3 V (ESP32 logic level); motor current is set over UART. The header pin order differs between makers: wire by pin name. 4. Motor connectors: pins 1-2 = one coil, pins 3-4 = the other coil. 5. A1 pin num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"
- note removed: "Battery voltage"
- note removed: "Both drivers share one single-wire UART: GPIO17 (TX) through R4, GPIO18 (RX) direct."
- note removed: "GPIO high = LED on. PWM sets the brightness."
- note removed: "Hand-unit socket (on the case)"
- note removed: "J1: female XT60 on the case, for the battery (LiFePO4 12.8 V 6 Ah with BMS) or a lab supply (12-14 V, current limit about 2 A). The battery is charged off the mount."
- note removed: "Power input, fuse, main switch"
- note removed: "U1 on a small TO-220 heatsink (tab = GND), about 1 W to dissipate. D1 stops the board's USB 5 V from feeding U1."
- note removed: "UART address 0 (MS1 = GND, MS2 = GND)"
- note removed: "UART address 1 (MS1 = 3V3, MS2 = GND)"
- note removed: "VBAT_SENSE = VBAT × 22 / 122 (14.6 V gives 2.63 V)"

Commit message: Remove the diode between the L7805 and the ESP32 board
The L7805 output goes straight to the board's 5V pin. Espressif lists
the board's USB ports and 5V pin as mutually exclusive power inputs,
so the docs and schematic now say not to connect USB while the breaker
is on, and to use Wi-Fi for logs and updates when the mount is powered.
The diode is listed under "Left out" for USB debugging with the motors
powered.

Co-Authored-By: Claude Opus 5.5 <noreply@anthropic.com>
Claude-Session: https://claude.ai/code/session_019gYbrjmddARBSj5u2J2ySh
Parts:
- removed BZ1: Buzzer, symbol Device:Buzzer
- removed CB1: Breaker switch, symbol Device:CircuitBreaker_1P
- removed D1: 1N5819, symbol Device:D_Schottky
- removed D4: blue, symbol Device:LED
- removed J2: Hand unit, 8 pins, symbol Connector_Generic:Conn_01x08
- removed R3: 10k, symbol Device:R
- added D3: red, symbol Device:LED
- added J1: XT60 female, symbol Connector_Generic:Conn_01x02
- added J5: ALT motor, symbol Connector_Generic:Conn_01x04
- added R7: 1k, symbol Device:R
- added SW2: E-stop (NC), symbol Switch:SW_Push_Open
- BZ1: renamed from R8; value 220 -> Buzzer; symbol Device:R -> Device:Buzzer
- CB1: renamed from J1; value XT60 female -> Breaker switch; symbol Connector_Generic:Conn_01x02 -> Device:CircuitBreaker_1P
- D4: renamed from D3; value red -> blue
- J2: renamed from SW2; value E-stop (NC) -> Hand unit, 8 pins; symbol Switch:SW_Push_Open -> Connector_Generic:Conn_01x08
- R3: renamed from J5; value ALT motor -> 10k; symbol Connector_Generic:Conn_01x04 -> Device:R
- R8: renamed from R7; value 1k -> 220
Connections:
- net +12V: now also CB1.2
- net +3V3: now also J2.2 (Pin_2), R3.1
- net +5V: now also U1.3 (OUT)
- net BTN1: now also J2.6 (Pin_6)
- net BTN2: now also J2.7 (Pin_7)
- net BTN3: now also J2.8 (Pin_8)
- net BUZZER: now also BZ1.1 (+)
- net DRV_EN: now also R3.2, SW2.2 (B); no longer J2.2 (B)
- net EN_OUT: now also SW2.1 (A); no longer J2.1 (A)
- net GND: now also BZ1.2 (-), J2.1 (Pin_1), D3.1 (K), J1.2 (Pin_2); no longer CB1.2 (Pin_2)
- net JOY_SW: now also J2.5 (Pin_5)
- net JOY_X: now also J2.3 (Pin_3)
- net JOY_Y: now also J2.4 (Pin_4)
- net LED_BLUE: now also R8.1; no longer BZ1.1
- net LED_RED: now also R7.1; no longer R8.1
- net at A3.11 (2B): now also J5.4 (Pin_4); no longer R3.4 (Pin_4)
- net at A3.12 (2A): now also J5.3 (Pin_3); no longer R3.3 (Pin_3)
- net at A3.13 (1A): now also J5.1 (Pin_1); no longer R3.1 (Pin_1)
- net at A3.14 (1B): now also J5.2 (Pin_2); no longer R3.2 (Pin_2)
- net at CB1.1: now also J1.1 (Pin_1)
- new net: D3.2 (A), R7.2
Other:
- note added: "U1 on a small TO-220 heatsink (tab = GND), about 1 W, near C6/C7, which serve as its input capacitors. CB1 on: keep the ESP32 board's USB unplugged. USB plugged in: keep CB1 off. The board's USB and 5V pin are not meant to supply power together."
- note removed: "U1 on a small TO-220 heatsink (tab = GND), about 1 W. Place it near C6/C7, which also serve as its input capacitors. D1 stops U1 and the board's USB 5 V from feeding each other."
- moved on the sheet: D4, R8

Commit message: Add a stripboard layout for the electronics, and a parts list
- electronics/star-track.kicad_pcb: 24 x 56 hole stripboard. Strips are
  B.Cu tracks with 54 cuts, wire links are board-only parts with joined
  pads, so DRC checks the board against the schematic (0 violations).
- Project footprints for the ESP32-S3-DevKitC-1 and the TMC2209 module.
- Pictures of the component side and the copper side.
- Schematic rev 5: GPIOs chosen to suit the stripboard, motor connector
  pins in module order, footprints assigned, case and hand-unit parts
  marked off the board.
- docs: stripboard section, new pin table, electronics parts list.
- Ignore KiCad local settings, locks and backups.

Co-Authored-By: Claude Opus 5.5 <noreply@anthropic.com>
Parts:
- A1: footprint (none) -> star-track:ESP32-S3-DevKitC-1_Socket
- A2, A3: footprint (none) -> star-track:TMC2209_StepStick_Socket
- C6, C7: footprint (none) -> Capacitor_THT:CP_Radial_D6.3mm_P2.50mm
- J4, J5: footprint (none) -> Connector_PinHeader_2.54mm:PinHeader_1x04_P2.54mm_Vertical
- R3: footprint (none) -> Resistor_THT:R_Axial_DIN0207_L6.3mm_D2.5mm_P7.62mm_Horizontal
- R7, R8: footprint (none) -> Resistor_THT:R_Axial_DIN0207_L6.3mm_D2.5mm_P10.16mm_Horizontal
- U1: footprint (none) -> Package_TO_SOT_THT:TO-220-3_Vertical
Connections:
- net ALT_DIR: now also A1.16 (GPIO10); no longer A1.20 (GPIO14)
- net ALT_STEP: now also A1.17 (GPIO11); no longer A1.19 (GPIO13)
- net AZ_DIR: now also A1.4 (GPIO4); no longer A1.18 (GPIO12)
- net AZ_STEP: now also A1.5 (GPIO5); no longer A1.17 (GPIO11)
- net BTN1: now also A1.29 (GPIO41); no longer A1.6 (GPIO6)
- net BTN2: now also A1.30 (GPIO40); no longer A1.7 (GPIO7)
- net BTN3: now also A1.31 (GPIO39); no longer A1.12 (GPIO8)
- net BUZZER: now also A1.20 (GPIO14); no longer A1.40 (GPIO21)
- net DRV_EN: now also A1.11 (GPIO18); no longer A1.15 (GPIO9)
- net EN_OUT: now also A1.15 (GPIO9); no longer A1.16 (GPIO10)
- net JOY_SW: now also A1.28 (GPIO42); no longer A1.5 (GPIO5)
- net LED_BLUE: now also A1.19 (GPIO13); no longer A1.9 (GPIO16)
- net LED_RED: now also A1.18 (GPIO12); no longer A1.8 (GPIO15)
- net at J4.1 (Pin_1): now also A2.14 (1B); no longer A2.13 (1A)
- net at J4.2 (Pin_2): now also A2.13 (1A); no longer A2.14 (1B)
- net at J5.1 (Pin_1): now also A3.14 (1B); no longer A3.13 (1A)
- net at J5.2 (Pin_2): now also A3.13 (1A); no longer A3.14 (1B)
Other:
- note added: "GPIO9 drives EN_OUT low to enable the drivers. E-stop pressed or ESP32 in reset: R3 pulls DRV_EN high and both drivers switch off. GPIO18 reads DRV_EN to detect it."
- note added: "Left free: GPIO0, 3, 45, 46 (strapping pins), GPIO19/20 (USB), GPIO35-37 (PSRAM on some boards), GPIO38 (RGB LED), GPIO43/44 (USB serial console)."
- note removed: "GPIO10 drives EN_OUT low to enable the drivers. E-stop pressed or ESP32 in reset: R3 pulls DRV_EN high and both drivers switch off. GPIO9 reads DRV_EN to detect it."
- note removed: "Left free: GPIO0, 3, 45, 46 (strapping pins), GPIO19/20 (USB), GPIO35-37 (PSRAM on some boards), GPIO43/44 (USB serial console)."

Commit message: Drop the buzzer; colour the stripboard pictures by net
- Remove BZ1 and its GPIO from the schematic, the stripboard and the
  docs. Feedback at the mount is the two LEDs. P2 keeps five pads.
- Stripboard pictures: one colour per net for the strips and the wire
  links, fixed colours for GND, +12V, +3V3 and +5V.

Co-Authored-By: Claude Opus 5.5 <noreply@anthropic.com>
Parts:
- removed BZ1: Buzzer, symbol Device:Buzzer
Connections:
- net BUZZER: no longer names the net of A1.20 (GPIO14)
- no-connect marks 26 -> 27
Other:
- note added: "GPIO high = LED on. PWM sets the brightness."
- note added: "LEDs (on the case)"
- note removed: "GPIO high = LED or buzzer on. PWM sets the LED brightness, or the tone of a passive buzzer."
- note removed: "LEDs and buzzer (on the case)"

Commit message: Replace the L7805 with a DC-DC converter, add a GPS module
- U1 is now a DC-DC step-down module set to 5 V, off the board on three
  wires (pads P5). The L7805 and its heatsink are gone.
- GPS module GY-GPS6MV2 (u-blox NEO-6M) on GPIO16/17, powered from 5 V,
  wired to pads P4. It gives the time and the site to the firmware.
- Motor cables are soldered into J4, J5.
- Stripboard pictures: the notes under the board are laid out in columns.
- docs: power, GPS, pins, power budget and parts list updated.

Co-Authored-By: Claude Opus 5.5 <noreply@anthropic.com>
Parts:
- removed J4: AZ motor, Connector_PinHeader_2.54mm:PinHeader_1x04_P2.54mm_Vertical, symbol Connector_Generic:Conn_01x04
- removed U1: L7805CV, Package_TO_SOT_THT:TO-220-3_Vertical, symbol Regulator_Linear:L7805
- added C7: 100µF 25V, Capacitor_THT:CP_Radial_D6.3mm_P2.50mm, symbol Device:C_Polarized
- added D3: red, symbol Device:LED
- added U2: GY-GPS6MV2, symbol Connector_Generic:Conn_01x04
- J4: renamed from C7; value 100µF 25V -> AZ motor; footprint Capacitor_THT:CP_Radial_D6.3mm_P2.50mm -> Connector_PinHeader_2.54mm:PinHeader_1x04_P2.54mm_Vertical; symbol Device:C_Polarized -> Connector_Generic:Conn_01x04
- U1: renamed from D3; value red -> DC-DC 5V module; symbol Device:LED -> Connector_Generic:Conn_01x03
Connections:
- net +12V: now also U1.1 (Pin_1), C7.1; no longer J4.1
- net +5V: now also U1.3 (Pin_3), U2.1 (Pin_1)
- net GND: now also U1.2 (Pin_2), C7.2, D3.1 (K), U2.4 (Pin_4); no longer J4.2, U1.1 (K)
- net at R7.2: now also D3.2 (A); no longer U1.2 (A)
- net GPS_TX: now reaches A1.10 (GPIO17)
- net GPS_TX: now also U2.3 (Pin_3)
- net GPS_RX: now reaches A1.9 (GPIO16)
- net GPS_RX: now also U2.2 (Pin_2)
- net at A2.14 (1B): now also J4.1 (Pin_1)
- net at A2.13 (1A): now also J4.2 (Pin_2)
- net at A2.12 (2A): now also J4.3 (Pin_3)
- net at A2.11 (2B): now also J4.4 (Pin_4)
- no-connect marks 27 -> 25
Other:
- note added: "GPS (on the case)"
- note added: "GPS module (u-blox NEO-6M): 1 VCC, 2 RX, 3 TX, 4 GND. VCC 3.3-5 V, 3.3 V logic, UART 9600 baud. Antenna towards the sky. Wired to pads P4."
- note added: "U1: DC-DC step-down module set to 5 V (1 VIN, 2 GND, 3 VOUT), off the board, wired to pads P5. CB1 on: keep the ESP32 board's USB unplugged. USB plugged in: keep CB1 off. The board's USB and 5V pin are not meant to supply power together."
- note removed: "U1 on a small TO-220 heatsink (tab = GND), about 1 W, near C6/C7, which serve as its input capacitors. CB1 on: keep the ESP32 board's USB unplugged. USB plugged in: keep CB1 off. The board's USB and 5V pin are not meant to supply power together."
